File: power_board/half_bridge.kicad_sch (KiCad schematic)
At the start: 24 parts, among them Q1 BSC0702LS, Q2 BSC0702LS, U5 UCC27282DRCR, U6 66565S0M3

Commit message: Complete all design, pass DRC
Parts:
- added TP37: VSS, esc-library:SMD_RH-5015, symbol Connector:TestPoint
- TP10: value TestPoint -> MOS_G_H
- TP11: value TestPoint -> DRIVE_H
- TP12: value TestPoint -> DRIVE_L
- TP13: value TestPoint -> PHASE_FB
- TP9: value TestPoint -> MOS_G_L
Connections:
- net VSS: now also TP37.1
Changed lines of the file:
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@@
+		)
+	)
+	(hierarchical_label "VSS"
+		(shape input)
+		(at 118.11 99.06 180)
+		(effects
+			(font
+				(size 1.27 1.27)
+			)
+			(justify right)
 		)
 	)
@@
 			)
 		)
-		(property "Value" "TestPoint"
+		(property "Value" "MOS_G_H"
 			(at 91.44 43.6879 0)
 			(effects
@@
 		(fields_autoplaced yes)
 		(property "Reference" "TP12"
-			(at 96.54 132.5879 0)
-			(effects
-				(font
-					(size 1.27 1.27)
-				)
-				(justify left)
-			)
-		)
-		(property "Value" "TestPoint"
-			(at 96.54 135.1279 0)
+			(at 96.52 132.5879 0)
+			(effects
+				(font
+					(size 1.27 1.27)
+				)
+				(justify left)
+			)
+		)
+		(property "Value" "DRIVE_L"
+			(at 96.52 135.1279 0)
 			(effects
 				(font
@@
 	(symbol
 		(lib_id "Connector:TestPoint")
+		(at 118.11 99.06 0)
+		(unit 1)
+		(exclude_from_sim no)
+		(in_bom yes)
+		(on_board yes)
+		(dnp no)
+		(fields_autoplaced yes)
+		(property "Reference" "TP37"
+			(at 120.65 94.4879 0)
+			(effects
+				(font
+					(size 1.27 1.27)
+				)
+				(justify left)
+			)
+		)
+		(property "Value" "VSS"
+			(at 120.65 97.0279 0)
+			(effects
+				(font
+					(size 1.27 1.27)
+				)
+				(justify left)
+			)
+		)
+		(property "Footprint" "esc-library:SMD_RH-5015"
+			(at 123.19 99.06 0)
+			(effects
+				(font
+					(size 1.27 1.27)
+				)
+				(hide yes)
+			)
+		)
+		(property "Datasheet" "~"
+			(at 123.19 99.06 0)
+			(effects
+				(font
+					(size 1.27 1.27)
+				)
+				(hide yes)
+			)
+		)
+		(property "Description" "test point"
+			(at 118.11 99.06 0)
+			(effects
+				(font
+					(size 1.27 1.27)
+				)
+				(hide yes)
+			)
+		)
+		(pin "1"
+		)
+		(instances
+			(project "power_board"
+				(path "/c786dd1f-c97f-4c1e-a27a-ac5828b3c50c/0fbb45d6-7cc5-4771-8820-af30fd089845"
+					(reference "TP38")
+					(unit 1)
+				)
+				(path "/c786dd1f-c97f-4c1e-a27a-ac5828b3c50c/38fb28ef-c920-476e-98e2-c5764b02e9b3"
+					(reference "TP37")
+					(unit 1)
+				)
+				(path "/c786dd1f-c97f-4c1e-a27a-ac5828b3c50c/74dd21af-da9a-49ef-aa54-e651b1250580"
+					(reference "TP39")
+					(unit 1)
+				)
+			)
+		)
+	)
+	(symbol
+		(lib_id "Connector:TestPoint")
 		(at 87.63 80.01 0)
 		(unit 1)
@@
 			)
 		)
-		(property "Value" "TestPoint"
+		(property "Value" "MOS_G_L"
 			(at 90.17 77.9779 0)
 			(effects
@@
 			)
 		)
-		(property "Value" "TestPoint"
+		(property "Value" "DRIVE_H"
 			(at 95.25 132.5879 0)
 			(effects
@@
 			)
 		)
-		(property "Value" "TestPoint"
+		(property "Value" "PHASE_FB"
 			(at 182.88 136.3979 0)
 			(effects
